File: esp_wifi_arduino.sch (KiCad schematic (older format))
At the start: 30 parts, among them CON1 AVR-ISP-6, IC1 ATMEGA328P-A, P1 CONN_15, P2 CONN_15, SW1 SW_PUSH, SW2 SW_PUSH, SW3 DIPSW4, U1 ADG3304, U2 ESP-WROOM-02, U3 NJM2391DL1-33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

Commit message: Create Footprint
Other:
- note added: "3.3V 1A"
- note added: "5V - 3.3V Convert\n"
- note added: "AVRISP"
- note added: "BOOT Mode"
Changed lines of the file:
@@
 $EndComp
 Text Label 6675 3450 0    60   ~ 0
+ArduinoRX33
+Text Label 6675 3550 0    60   ~ 0
 ArduinoTX33
-Text Label 6675 3550 0    60   ~ 0
-ArduinoRX33
 Text Label 9475 5550 0    60   ~ 0
 ArduinoTX33
@@
 Arduino nano compatible.
 Connection ~ 1750 1950
+Text Notes 5250 3200 0    60   ~ 0
+5V - 3.3V Convert\n
+Text Notes 3900 5000 0    60   ~ 0
+3.3V 1A
+Text Notes 5250 4850 0    60   ~ 0
+BOOT Mode
+Text Notes 7900 1650 0    60   ~ 0
+AVRISP
 $EndSCHEMATC

Commit message: Circuit Create
Parts:
- removed CON1: AVR-ISP-6, AVR-ISP-6, symbol AVR-ISP-6
- added P3, P4: CONN_1, ~, symbol CONN_1
Connections:
- wire segments 153 -> 155
Changed lines of the file:
@@
 LIBS:valves
 LIBS:kamiya_components
+LIBS:esp_wifi_arduino-cache
 EELAYER 27 0
 EELAYER END
@@
 Sheet 1 1
 Title "Arduino with ESP-WROOM-02"
-Date "24 oct 2015"
+Date "25 oct 2015"
 Rev "A"
 Comp "Asumono-LAB"
@@
 F 3 "" H 3175 2750 60  0000 C CNN
 	1    3175 2750
-	1    0    0    -1
-$EndComp
-$Comp
-L AVR-ISP-6 CON1
-U 1 1 562B43E3
-P 8475 2025
-F 0 "CON1" H 8395 2265 50  0000 C CNN
-F 1 "AVR-ISP-6" H 8235 1795 50  0000 L BNN
-F 2 "AVR-ISP-6" V 7955 2065 50  0001 C CNN
-F 3 "" H 8475 2025 60  0000 C CNN
-	1    8475 2025
 	1    0    0    -1
 $EndComp
@@
 Text Notes 7900 1650 0    60   ~ 0
 AVRISP
+Connection ~ 9525 5150
+Connection ~ 10125 5150
+Connection ~ 7775 2125
+Connection ~ 7175 2125
+$Comp
+L GND #PWR035
+U 1 1 562CAD09
+P 4075 4725
+F 0 "#PWR035" H 4075 4725 30  0001 C CNN
+F 1 "GND" H 4075 4655 30  0001 C CNN
+F 2 "" H 4075 4725 60  0000 C CNN
+F 3 "" H 4075 4725 60  0000 C CNN
+	1    4075 4725
+	1    0    0    -1
+$EndComp
+$Comp
+L CONN_1 P3
+U 1 1 562CAD21
+P 4075 4475
+F 0 "P3" H 4155 4475 40  0000 L CNN
+F 1 "CONN_1" H 4075 4530 30  0001 C CNN
+F 2 "~" H 4075 4475 60  0000 C CNN
+F 3 "~" H 4075 4475 60  0000 C CNN
+	1    4075 4475
+	0    -1   -1   0
+$EndComp
+$Comp
+L CONN_1 P4
+U 1 1 562CAD2E
+P 4175 4475
+F 0 "P4" H 4255 4475 40  0000 L CNN
+F 1 "CONN_1" H 4175 4530 30  0001 C CNN
+F 2 "~" H 4175 4475 60  0000 C CNN
+F 3 "~" H 4175 4475 60  0000 C CNN
+	1    4175 4475
+	0    -1   -1   0
+$EndComp
+Wire Wire Line
+	4075 4625 4075 4725
+Wire Wire Line
+	4175 4625 4075 4625
+Connection ~ 4175 4625
+Connection ~ 4075 4625
 $EndSCHEMATC

Commit message: Before Rev.B
Parts:
- C1, C10, C2, C3, C4, C5, C6, C7, C8, C9: symbol C -> C-RESCUE-esp_wifi_arduino
- D1, D2: symbol LED -> LED-RESCUE-esp_wifi_arduino
- IC1: symbol ATMEGA328P-A -> ATMEGA328P-A-RESCUE-esp_wifi_arduino
- R1, R2, R3, R4, R5, R6, R7: symbol R -> R-RESCUE-esp_wifi_arduino
Changed lines of the file:
@@
 EESchema Schematic File Version 2
+LIBS:esp_wifi_arduino-rescue
 LIBS:power
 LIBS:device
@@
 LIBS:memory
 LIBS:xilinx
-LIBS:special
 LIBS:microcontrollers
 LIBS:dsp
@@
 LIBS:contrib
 LIBS:valves
-LIBS:kamiya_components
 LIBS:esp_wifi_arduino-cache
-EELAYER 27 0
+EELAYER 25 0
 EELAYER END
 $Descr A4 11693 8268
@@
 $EndComp
 $Comp
-L ATMEGA328P-A IC1
+L ATMEGA328P-A-RESCUE-esp_wifi_arduino IC1
 U 1 1 562B43CA
 P 3175 2750
@@
 $EndComp
 $Comp
-L C C8
+L C-RESCUE-esp_wifi_arduino C8
 U 1 1 562B45B8
 P 2575 5425
@@
 $EndComp
 $Comp
-L C C9
+L C-RESCUE-esp_wifi_arduino C9
 U 1 1 562B45C5
 P 4025 5425
@@
 $EndComp
 $Comp
-L +3.3V #PWR01
+L +3.3V-RESCUE-esp_wifi_arduino #PWR01
 U 1 1 562B463A
 P 4125 5175
@@
 $EndComp
 $Comp
-L GND #PWR03
+L GND-RESCUE-esp_wifi_arduino #PWR03
 U 1 1 562B4658
 P 3275 5875
@@
 $EndComp
 $Comp
-L +3.3V #PWR06
+L +3.3V-RESCUE-esp_wifi_arduino #PWR06
 U 1 1 562B4C64
 P 6425 3300
@@
 $EndComp
 $Comp
-L GND #PWR07
+L GND-RESCUE-esp_wifi_arduino #PWR07
 U 1 1 562B4C79
 P 4875 4325
@@
 $EndComp
 $Comp
-L C C2
+L C-RESCUE-esp_wifi_arduino C2
 U 1 1 562B4D1C
 P 1600 1950
@@
 $EndComp
 $Comp
-L C C1
+L C-RESCUE-esp_wifi_arduino C1
 U 1 1 562B4D29
 P 1450 1850
@@
 $EndComp
 $Comp
-L GND #PWR09
+L GND-RESCUE-esp_wifi_arduino #PWR09
 U 1 1 562B4DC1
 P 1450 2500
@@
 $EndComp
 $Comp
-L C C3
+L C-RESCUE-esp_wifi_arduino C3
 U 1 1 562B4DE7
 P 1750 2150
@@
 $EndComp
 $Comp
-L GND #PWR010
+L GND-RESCUE-esp_wifi_arduino #PWR010
 U 1 1 562B4F62
 P 2125 4050
@@
 $EndComp
 $Comp
-L R R4
+L R-RESCUE-esp_wifi_arduino R4
 U 1 1 562B4FF1
 P 9525 4850
@@
 $EndComp
 $Comp
-L +3.3V #PWR011
+L +3.3V-RESCUE-esp_wifi_arduino #PWR011
 U 1 1 562B5060
 P 9525 4550
@@
 $EndComp
 $Comp
-L GND #PWR012
+L GND-RESCUE-esp_wifi_arduino #PWR012
 U 1 1 562B509D
 P 7175 6225
@@
 $EndComp
 $Comp
-L GND #PWR013
+L GND-RESCUE-esp_wifi_arduino #PWR013
 U 1 1 562B50D2
 P 9275 5400
@@
 $EndComp
 $Comp
-L R R3
+L R-RESCUE-esp_wifi_arduino R3
 U 1 1 562B51A9
 P 6625 4850
@@
 $EndComp
 $Comp
-L R R5
+L R-RESCUE-esp_wifi_arduino R5
 U 1 1 562B5202
 P 6475 5000
@@
 $EndComp
 $Comp
-L R R6
+L R-RESCUE-esp_wifi_arduino R6
 U 1 1 562B5208
 P 6325 5150
@@
 $EndComp
 $Comp
-L R R7
+L R-RESCUE-esp_wifi_arduino R7
 U 1 1 562B520E
 P 6175 5300
@@
 $EndComp
 $Comp
-L +3.3V #PWR014
+L +3.3V-RESCUE-esp_wifi_arduino #PWR014
 U 1 1 562B5214
 P 7175 4800
@@
 $EndComp
 $Comp
-L +3.3V #PWR015
+L +3.3V-RESCUE-esp_wifi_arduino #PWR015
 U 1 1 562B5260
 P 6625 4550
@@
 $EndComp
 $Comp
-L GND #PWR016
+L GND-RESCUE-esp_wifi_arduino #PWR016
 U 1 1 562B536B
 P 4875 5750
@@
 $EndComp
 $Comp
-L GND #PWR017
+L GND-RESCUE-esp_wifi_arduino #PWR017
 U 1 1 562B5495
 P 9275 4900
@@
 $EndComp
 $Comp
-L GND #PWR018
+L GND-RESCUE-esp_wifi_arduino #PWR018
 U 1 1 562B54E9
 P 10225 5200
@@
 $EndComp
 $Comp
-L R R1
+L R-RESCUE-esp_wifi_arduino R1
 U 1 1 562B57C2
 P 5325 2150
@@
 $EndComp
 $Comp
-L LED D1
+L LED-RESCUE-esp_wifi_arduino D1
 U 1 1 562B5824
 P 5875 2150
@@
 $EndComp
 $Comp
-L GND #PWR019
+L GND-RESCUE-esp_wifi_arduino #PWR019
 U 1 1 562B5831
 P 6175 2250
@@
 $EndComp
 $Comp
-L C C4
+L C-RESCUE-esp_wifi_arduino C4
 U 1 1 562B5CD6
 P 4825 2800
@@
 $EndComp
 $Comp
-L C C5
+L C-RESCUE-esp_wifi_arduino C5
 U 1 1 562B5CF7
 P 5425 2800
@@
 $EndComp
 $Comp
-L GND #PWR020
+L GND-RESCUE-esp_wifi_arduino #PWR020
 U 1 1 562B5CFD
 P 4825 3050
@@
 $EndComp
 $Comp
-L GND #PWR021
+L GND-RESCUE-esp_wifi_arduino #PWR021
 U 1 1 562B5D6B
 P 5425 3050
@@
 $EndComp
 $Comp
-L GND #PWR023
+L GND-RESCUE-esp_wifi_arduino #PWR023
 U 1 1 562B67E7
 P 8975 2150
@@
 $EndComp
 $Comp
-L R R2
+L R-RESCUE-esp_wifi_arduino R2
 U 1 1 562B6D94
 P 2950 4625
@@
 $EndComp
 $Comp
-L LED D2
+L LED-RESCUE-esp_wifi_arduino D2
 U 1 1 562B6D9A
 P 3500 4625
@@
 $EndComp
 $Comp
-L GND #PWR024
+L GND-RESCUE-esp_wifi_arduino #PWR024
 U 1 1 562B6DA0
 P 3800 4725
@@
 $EndComp
 $Comp
-L GND #PWR026
+L GND-RESCUE-esp_wifi_arduino #PWR026
 U 1 1 562B7055
 P 7125 2175
@@
 D12
 $Comp
-L GND #PWR027
+L GND-RESCUE-esp_wifi_arduino #PWR027
 U 1 1 562B7319
 P 7400 3000
@@
 A0
 $Comp
-L +3.3V #PWR028
+L +3.3V-RESCUE-esp_wifi_arduino #PWR028
 U 1 1 562B76DE
 P 9250 3925
@@
 $EndComp
 $Comp
-L GND #PWR031
+L GND-RESCUE-esp_wifi_arduino #PWR031
 U 1 1 562B76F0
 P 9350 2775
@@
 $EndComp
 $Comp
-L +3.3V #PWR033
+L +3.3V-RESCUE-esp_wifi_arduino #PWR033
 U 1 1 562B7C34
 P 4775 3750
@@
 $EndComp
 $Comp
-L C C6
+L C-RESCUE-esp_wifi_arduino C6
 U 1 1 562B7CE0
 P 4575 4025
@@
 $EndComp
 $Comp
-L C C7
+L C-RESCUE-esp_wifi_arduino C7
 U 1 1 562B7A9D
 P 4775 4025
@@
 	4575 3750 4575 3825
 $Comp
-L C C10
+L C-RESCUE-esp_wifi_arduino C10
 U 1 1 562B8108
 P 7025 5925
@@
 $EndComp
 $Comp
-L +3.3V #PWR034
+L +3.3V-RESCUE-esp_wifi_arduino #PWR034
 U 1 1 562B81D7
 P 7025 5700
@@
 Connection ~ 7175 2125
 $Comp
-L GND #PWR035
+L GND-RESCUE-esp_wifi_arduino #PWR035
 U 1 1 562CAD09
 P 4075 4725

Commit message: PCB Layout
Parts:
- removed D1: LED, ~, symbol LED-RESCUE-esp_wifi_arduino
- removed P1, P2: CONN_15, ~, symbol CONN_15
- removed P3, P4: CONN_1, ~, symbol CONN_1
- removed R1: R, ~, symbol R-RESCUE-esp_wifi_arduino
- added P1, P2: CONN_01X15, Pin_Headers:Pin_Header_Straight_1x15, symbol CONN_01X15
- added P5, P6: CONN_01X04, Pin_Headers:Pin_Header_Straight_1x04, symbol CONN_01X04
- added S1: RX_SEL, kamiya:ALPS_SSSS213202(SlideSW), symbol SEL
- added S2: TX_SEL, kamiya:ALPS_SSSS213202(SlideSW), symbol SEL
- added S3: EN_SEL, kamiya:ALPS_SSSS213202(SlideSW), symbol SEL
- C1, C10, C2, C3, C4, C5, C6, C7, C8, C9, D2, R2, R3, R4, R5, R6, R7: footprint ~ -> kamiya:HANDSOL_0603
- IC1: footprint TQFP32 -> hastech:TQFP32-08
- SW1, SW2: footprint ~ -> kamiya:ALPS_SW_SKRPACE010
- SW3: footprint (none) -> kamiya:OTAX_DIPSW4
- U1: footprint (none) -> kamiya:AD_TSSOP-14(0.65)
- U2: footprint ~ -> kamiya:ESP_WROOM_02
- U3: footprint ~ -> kamiya:TO-252-3
- X1: footprint ~ -> kamiya:XTAL_HC-49
Connections:
- net labels added: ESP_RX, ESP_TX, IO12, IO13, IO14, IO16, IO4, IO5
- net labels removed: ArduinoRX33, ArduinoTX33
- wire segments 155 -> 202
- no-connect marks 0 -> 5
Other:
- note added: "Arduino Pro Mini compatible."
- note added: "ESP-WROOM-02 GPIO"
- note removed: "Arduino nano compatible."
- moved on the sheet: C1, C10, C2, C3, C4, C5, C6, C7, C8, C9, D2, IC1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

Commit message: Draw Pattern
Parts:
- removed S3: EN_SEL, kamiya:ALPS_SSSS213202(SlideSW), symbol SEL
- added SW4: SWITCH_INV, ~, symbol SWITCH_INV
Connections:
- wire segments 202 -> 178
Changed lines of the file:
@@
 $EndComp
 $Comp
-L GND-RESCUE-esp_wifi_arduino #PWR019
+L GND-RESCUE-esp_wifi_arduino #PWR018
 U 1 1 562B5CFD
 P 4525 3875
-F 0 "#PWR019" H 4525 3875 30  0001 C CNN
+F 0 "#PWR018" H 4525 3875 30  0001 C CNN
 F 1 "GND" H 4525 3805 30  0001 C CNN
 F 2 "" H 4525 3875 60  0000 C CNN
@@
 $EndComp
 $Comp
-L GND-RESCUE-esp_wifi_arduino #PWR020
+L GND-RESCUE-esp_wifi_arduino #PWR019
 U 1 1 562B5D6B
 P 5125 3875
-F 0 "#PWR020" H 5125 3875 30  0001 C CNN
+F 0 "#PWR019" H 5125 3875 30  0001 C CNN
 F 1 "GND" H 5125 3805 30  0001 C CNN
 F 2 "" H 5125 3875 60  0000 C CNN
@@
 RESET
 $Comp
-L +5V #PWR021
+L +5V #PWR020
 U 1 1 562B67E1
 P 9725 5750
-F 0 "#PWR021" H 9725 5840 20  0001 C CNN
+F 0 "#PWR020" H 9725 5840 20  0001 C CNN
 F 1 "+5V" H 9725 5840 30  0000 C CNN
 F 2 "" H 9725 5750 60  0000 C CNN
@@
 $EndComp
 $Comp
-L GND-RESCUE-esp_wifi_arduino #PWR022
+L GND-RESCUE-esp_wifi_arduino #PWR021
 U 1 1 562B67E7
 P 9725 6025
-F 0 "#PWR022" H 9725 6025 30  0001 C CNN
+F 0 "#PWR021" H 9725 6025 30  0001 C CNN
 F 1 "GND" H 9725 5955 30  0001 C CNN
 F 2 "" H 9725 6025 60  0000 C CNN
@@
 $EndComp
 $Comp
-L GND-RESCUE-esp_wifi_arduino #PWR023
+L GND-RESCUE-esp_wifi_arduino #PWR022
 U 1 1 562B6DA0
 P 7150 3925
-F 0 "#PWR023" H 7150 3925 30  0001 C CNN
+F 0 "#PWR022" H 7150 3925 30  0001 C CNN
 F 1 "GND" H 7150 3855 30  0001 C CNN
 F 2 "" H 7150 3925 60  0000 C CNN
@@
 $EndComp
 $Comp
-L +5V #PWR024
+L +5V #PWR023
 U 1 1 562B6DA9
 P 5775 3800
-F 0 "#PWR024" H 5775 3890 20  0001 C CNN
+F 0 "#PWR023" H 5775 3890 20  0001 C CNN
 F 1 "+5V" H 5775 3890 30  0000 C CNN
 F 2 "" H 5775 3800 60  0000 C CNN
@@
 $EndComp
 $Comp
-L GND-RESCUE-esp_wifi_arduino #PWR025
+L GND-RESCUE-esp_wifi_arduino #PWR024
 U 1 1 562B7055
 P 7875 6050
-F 0 "#PWR025" H 7875 6050 30  0001 C CNN
+F 0 "#PWR024" H 7875 6050 30  0001 C CNN
 F 1 "GND" H 7875 5980 30  0001 C CNN
 F 2 "" H 7875 6050 60  0000 C CNN
@@
 D12
 $Comp
-L GND-RESCUE-esp_wifi_arduino #PWR026
+L GND-RESCUE-esp_wifi_arduino #PWR025
 U 1 1 562B7319
 P 8650 3400
-F 0 "#PWR026" H 8650 3400 30  0001 C CNN
+F 0 "#PWR025" H 8650 3400 30  0001 C CNN
 F 1 "GND" H 8650 3330 30  0001 C CNN
 F 2 "" H 8650 3400 60  0000 C CNN
@@
 A0
 $Comp
-L +3.3V-RESCUE-esp_wifi_arduino #PWR027
+L +3.3V-RESCUE-esp_wifi_arduino #PWR026
 U 1 1 562B76DE
 P 9875 4325
-F 0 "#PWR027" H 9875 4285 30  0001 C CNN
+F 0 "#PWR026" H 9875 4285 30  0001 C CNN
 F 1 "+3.3V" H 9875 4435 30  0000 C CNN
 F 2 "" H 9875 4325 60  0000 C CNN
@@
 $EndComp
 $Comp
-L +5V #PWR028
+L +5V #PWR027
 U 1 1 562B76E4
 P 9850 3000
-F 0 "#PWR028" H 9850 3090 20  0001 C CNN
+F 0 "#PWR027" H 9850 3090 20  0001 C CNN
 F 1 "+5V" H 9850 3090 30  0000 C CNN
 F 2 "" H 9850 3000 60  0000 C CNN
@@
 $EndComp
 $Comp
-L +5V #PWR029
+L +5V #PWR028
 U 1 1 562B76EA
 P 9850 3325
-F 0 "#PWR029" H 9850 3415 20  0001 C CNN
+F 0 "#PWR028" H 9850 3415 20  0001 C CNN
 F 1 "+5V" H 9850 3415 30  0000 C CNN
 F 2 "" H 9850 3325 60  0000 C CNN
@@
 $EndComp
 $Comp
-L GND-RESCUE-esp_wifi_arduino #PWR030
+L GND-RESCUE-esp_wifi_arduino #PWR029
 U 1 1 562B76F0
 P 9975 3175
-F 0 "#PWR030" H 9975 3175 30  0001 C CNN
+F 0 "#PWR029" H 9975 3175 30  0001 C CNN
 F 1 "GND" H 9975 3105 30  0001 C CNN
 F 2 "" H 9975 3175 60  0000 C CNN
@@
 $EndComp
 $Comp
-L +5V #PWR031
+L +5V #PWR030
 U 1 1 562B7AC7
 P 10300 2050
-F 0 "#PWR031" H 10300 2140 20  0001 C CNN
+F 0 "#PWR030" H 10300 2140 20  0001 C CNN
 F 1 "+5V" H 10300 2160 30  0000 C CNN
 F 2 "" H 10300 2050 60  0000 C CNN
@@
 $EndComp
 $Comp
-L +3.3V-RESCUE-esp_wifi_arduino #PWR032
+L +3.3V-RESCUE-esp_wifi_arduino #PWR031
 U 1 1 562B7C34
 P 10100 2050
-F 0 "#PWR032" H 10100 2010 30  0001 C CNN
+F 0 "#PWR031" H 10100 2010 30  0001 C CNN
 F 1 "+3.3V" H 10100 2160 30  0000 C CNN
 F 2 "" H 10100 2050 60  0000 C CNN
@@
 $EndComp
 $Comp
-L +3.3V-RESCUE-esp_wifi_arduino #PWR033
+L +3.3V-RESCUE-esp_wifi_arduino #PWR032
 U 1 1 562B81D7
 P 3225 6650
-F 0 "#PWR033" H 3225 6610 30  0001 C CNN
+F 0 "#PWR032" H 3225 6610 30  0001 C CNN
 F 1 "+3.3V" H 3225 6760 30  0000 C CNN
 F 2 "" H 3225 6650 60  0000 C CNN
@@
 $EndComp
 $Comp
-L SEL S3
-U 1 1 565B9EEA
-P 7725 2325
-F 0 "S3" H 8000 2500 60  0000 C CNN
-F 1 "EN_SEL" H 7650 2500 60  0000 C CNN
-F 2 "kamiya:ALPS_SSSS213202(SlideSW)" H 7725 2325 60  0001 C CNN
-F 3 "" H 7725 2325 60  0000 C CNN
-	1    7725 2325
-	-1   0    0    1
-$EndComp
-$Comp
-L +5V #PWR034
+L +5V #PWR033
 U 1 1 565BAAFD
-P 7100 2275
-F 0 "#PWR034" H 7100 2365 20  0001 C CNN
-F 1 "+5V" H 7100 2365 30  0000 C CNN
-F 2 "" H 7100 2275 60  0000 C CNN
-F 3 "" H 7100 2275 60  0000 C CNN
-	1    7100 2275
+P 7100 2175
+F 0 "#PWR033" H 7100 2265 20  0001 C CNN
+F 1 "+5V" H 7100 2265 30  0000 C CNN
+F 2 "" H 7100 2175 60  0000 C CNN
+F 3 "" H 7100 2175 60  0000 C CNN
+	1    7100 2175
 	-1   0    0    -1
 $EndComp
 $Comp
-L GND-RESCUE-esp_wifi_arduino #PWR035
+L GND-RESCUE-esp_wifi_arduino #PWR034
 U 1 1 565BB608
 P 7100 2525
-F 0 "#PWR035" H 7100 2525 30  0001 C CNN
+F 0 "#PWR034" H 7100 2525 30  0001 C CNN
 F 1 "GND" H 7100 2455 30  0001 C CNN
 F 2 "" H 7100 2525 60  0000 C CNN
@@
 $EndComp
 Wire Wire Line
-	5525 4375 5775 4375
-Wire Wire Line
-	5775 4375 5925 4375
-Wire Wire Line
-	5925 4375 6025 4375
+	5525 4375 6025 4375
 Wire Wire Line
 	5925 4425 5925 4375
@@
 	5925 4825 5925 4925
 Wire Wire Line
-	5925 4925 6625 4925
-Wire Wire Line
-	6625 4925 7375 4925
+	5925 4925 7375 4925
 Wire Wire Line
 	7375 4925 7375 4825
 Connection ~ 6625 4925
 Wire Wire Line
-	7225 4375 7375 4375
-Wire Wire Line
-	7375 4375 7475 4375
+	7225 4375 7475 4375
 Wire Wire Line
 	7375 4375 7375 4425
@@
 	9950 2250 10000 2250
 Wire Wire Line
-	10000 2250 10000 2525
-Wire Wire Line
-	10000 2525 10000 2625
+	10000 2250 10000 2625
 Wire Wire Line
 	9950 1750 10250 1750
@@
 	1150 2275 1150 2475
 Wire Wire Line
-	1150 2475 1300 2475
-Wire Wire Line
-	1300 2475 1975 2475
-Wire Wire Line
-	1300 2575 1450 2575
-Wire Wire Line
-	1450 2575 1975 2575
+	1150 2475 1975 2475
+Wire Wire Line
+	1300 2575 1975 2575
 Wire Wire Line
 	1300 2575 1300 2475
@@
 	1300 2975 1150 2975
 Wire Wire Line
-	1150 2875 1150 2975
-Wire Wire Line
-	1150 2975 1150 3175
-Wire Wire Line
-	1150 3175 1150 3325
+	1150 2875 1150 3325
 Connection ~ 1150 2975
 Wire Wire Line
@@
 	1975 4575 1825 4575
 Wire Wire Line
-	1825 4575 1825 4675
-Wire Wire Line
-	1825 4675 1825 4775
-Wire Wire Line
-	1825 4775 1825 4875
+	1825 4575 1825 4875
 Wire Wire Line
 	1975 4675 1825 4675
@@
 	3425 6600 3375 6600
 Wire Wire Line
-	3375 6600 3375 7075
-Wire Wire Line
-	3375 7075 3375 7175
+	3375 6600 3375 7175
 Wire Wire Line
 	5375 6300 5475 6300
@@
 	5475 6300 5475 6350
 Wire Wire Line
-	2325 6500 2375 6500
-Wire Wire Line
-	2375 6500 3425 6500
+	2325 6500 3425 6500
 Wire Wire Line
 	3425 6400 2925 6400
@@
 	2925 6400 2925 6350
 Wire Wire Line
-	2925 6350 2525 6350
-Wire Wire Line
-	2525 6350 2325 6350
+	2925 6350 2325 6350
 Wire Wire Line
 	3425 6300 2975 6300
@@
 	2975 6300 2975 6200
 Wire Wire Line
-	2975 6200 2675 6200
-Wire Wire Line
-	2675 6200 2325 6200
+	2975 6200 2325 6200
 Wire Wire Line
 	3425 5900 2975 5900
@@
 	2975 5900 2975 6050
 Wire Wire Line
-	2975 6050 2825 6050
-Wire Wire Line
-	2825 6050 2325 6050
+	2975 6050 2325 6050
 Wire Wire Line
 	3375 5750 3375 5800
@@
 	2825 5550 2825 5500
 Wire Wire Line
-	2375 5550 2525 5550
-Wire Wire Line
-	2525 5550 2675 5550
-Wire Wire Line
-	2675 5550 2825 5550
+	2375 5550 2825 5550
 Wire Wire Line
 	2675 5550 2675 5700
@@
 	1075 6500 1175 6500
 Wire Wire Line
-	1075 6050 1075 6200
-Wire Wire Line
-	1075 6200 1075 6350
-Wire Wire Line
-	1075 6350 1075 6500
-Wire Wire Line
-	1075 6500 1075 6700
+	1075 6050 1075 6700
 Wire Wire Line
 	1175 6350 1075 6350
@@
 	5125 3825 5125 3875
 Wire Wire Line
-	5125 3075 5125 3375
-Wire Wire Line
-	5125 3375 5125 3425
-Wire Wire Line
-	4525 3175 4525 3375
-Wire Wire Line
-	4525 3375 4525 3425
+	5125 3075 5125 3425
+Wire Wire Line
+	4525 3175 4525 3425
 Wire Wire Line
 	4525 3175 3875 3175
@@
 	9875 4350 9875 4325
 Wire Wire Line
-	10000 2525 10100 2525
-Wire Wire Line
-	10100 2525 10300 2525
+	10000 2525 10300 2525
 Connection ~ 10000 2525
 Wire Wire Line
@@
 	8325 1950 8175 1950
 Wire Wire Line
-	7100 2275 7100 2325
-Wire Wire Line
-	7100 2325 7175 2325
+	7100 2175 7100 2225
+Wire Wire Line
+	7100 2225 7175 2225
 Wire Wire Line
 	7175 2425 7100 2425
@@
 NoConn ~ 9950 2050
 $Comp
-L PWR_FLAG #FLG036
+L PWR_FLAG #FLG035
 U 1 1 565D8F5F
 P 5525 4375
-F 0 "#FLG036" H 5525 4470 50  0001 C CNN
+F 0 "#FLG035" H 5525 4470 50  0001 C CNN
 F 1 "PWR_FLAG" H 5525 4555 50  0000 C CNN
 F 2 "" H 5525 4375 60  0000 C CNN
@@
 Connection ~ 5775 4375
 NoConn ~ 5375 6000
+$Comp
+L SWITCH_INV SW4
+U 1 1 565B1479
+P 7675 2325
+F 0 "SW4" H 7475 2475 50  0000 C CNN
+F 1 "SWITCH_INV" H 7525 2175 50  0000 C CNN
+F 2 "~" H 7675 2325 60  0000 C CNN
+F 3 "~" H 7675 2325 60  0000 C CNN
+	1    7675 2325
+	-1   0    0    1
+$EndComp
 $EndSCHEMATC

Commit message: Create Production File
Other:
- moved on the sheet: P5, P6
Changed lines of the file:
@@
 Sheet 1 1
 Title "Arduino with ESP-WROOM-02"
-Date "29 nov 2015"
+Date "30 nov 2015"
 Rev "A"
 Comp "Asumono-LAB"
@@
 Text Notes 1450 5800 0    60   ~ 0
 BOOT Mode
-Text Notes 8650 5525 0    60   ~ 0
+Text Notes 8650 5650 0    60   ~ 0
 AVRISP
 Text Label 7025 1750 2    60   ~ 0
@@
 	8350 2325 8175 2325
 Wire Wire Line
+	9575 5200 9800 5200
+Wire Wire Line
+	9575 5100 9800 5100
+Wire Wire Line
+	9575 5000 9800 5000
+Wire Wire Line
+	8975 5200 8750 5200
+Wire Wire Line
+	8975 5100 8750 5100
+Wire Wire Line
 	8975 5000 8750 5000
-Wire Wire Line
-	8975 5100 8750 5100
-Wire Wire Line
-	8975 5200 8750 5200
-Wire Wire Line
-	9575 5000 9800 5000
-Wire Wire Line
-	9575 5100 9800 5100
-Wire Wire Line
-	9575 5200 9800 5200
 Wire Wire Line
 	5625 5800 5625 5875
@@
 Text Label 3275 6200 0    60   ~ 0
 IO13
-Text Label 9775 5200 2    60   ~ 0
+Text Label 8775 5000 0    60   ~ 0
 IO14
-Text Label 8750 5200 0    60   ~ 0
+Text Label 9800 5000 2    60   ~ 0
 IO12
-Text Label 8750 5300 0    60   ~ 0
+Text Label 9800 4900 2    60   ~ 0
 IO13
-Text Label 8750 5000 0    60   ~ 0
+Text Label 9800 5200 2    60   ~ 0
 IO4
-Text Label 8750 5100 0    60   ~ 0
+Text Label 9800 5100 2    60   ~ 0
 IO5
-Text Label 9775 5300 2    60   ~ 0
+Text Label 8775 4900 0    60   ~ 0
 IO16
 $Comp
 L CONN_01X04 P5
 U 1 1 565CD625
-P 9175 5150
-F 0 "P5" H 9175 5400 50  0000 C CNN
-F 1 "CONN_01X04" V 9275 5150 50  0000 C CNN
-F 2 "Pin_Headers:Pin_Header_Straight_1x04" H 9175 5150 60  0001 C CNN
-F 3 "" H 9175 5150 60  0000 C CNN
-	1    9175 5150
-	1    0    0    -1
+P 9375 5050
+F 0 "P5" H 9375 5300 50  0000 C CNN
+F 1 "CONN_01X04" V 9475 5050 50  0000 C CNN
+F 2 "Pin_Headers:Pin_Header_Straight_1x04" H 9375 5050 60  0001 C CNN
+F 3 "" H 9375 5050 60  0000 C CNN
+	1    9375 5050
+	-1   0    0    1
 $EndComp
 $Comp
 L CONN_01X04 P6
 U 1 1 565CD6C2
-P 9375 5150
-F 0 "P6" H 9375 5400 50  0000 C CNN
-F 1 "CONN_01X04" V 9475 5150 50  0000 C CNN
-F 2 "Pin_Headers:Pin_Header_Straight_1x04" H 9375 5150 60  0001 C CNN
-F 3 "" H 9375 5150 60  0000 C CNN
-	1    9375 5150
-	-1   0    0    1
-$EndComp
-Wire Wire Line
-	8975 5300 8750 5300
-Wire Wire Line
-	9575 5300 9800 5300
-Text Notes 8775 4825 0    60   ~ 0
+P 9175 5050
+F 0 "P6" H 9175 5300 50  0000 C CNN
+F 1 "CONN_01X04" V 9275 5050 50  0000 C CNN
+F 2 "Pin_Headers:Pin_Header_Straight_1x04" H 9175 5050 60  0001 C CNN
+F 3 "" H 9175 5050 60  0000 C CNN
+	1    9175 5050
+	1    0    0    -1
+$EndComp
+Wire Wire Line
+	9575 4900 9800 4900
+Wire Wire Line
+	8975 4900 8750 4900
+Text Notes 8800 4750 0    60   ~ 0
 ESP-WROOM-02 GPIO
 Text Label 10250 1750 2    60   ~ 0
@@
 Text Label 10250 1850 2    60   ~ 0
 ESP_RX
-Text Label 9600 5000 0    60   ~ 0
+Text Label 8950 5200 2    60   ~ 0
 ESP_TX
-Text Label 9600 5100 0    60   ~ 0
+Text Label 8950 5100 2    60   ~ 0
 ESP_RX
 NoConn ~ 8500 1950
